File: eagle/3phasecntrl-rev0.sch (EAGLE design)
At the start: 66 parts, among them IC3 ATXmega32A4U, IC4 LD1117S50, IC6 LD1117S33, T1 BC847, T2 BC847, U1 LM5008MM

Commit message: Added farnell parts to eagledb file, BOM.
Parts:
- C2: value 100 -> 100n
- C5: value 33u/25V -> 68u/25V
- C7: value 100n? -> 100n
- D1: value BAT46WH -> SS110B
- F1: value (none) -> 140mA
- R12: value 1k? -> 1k
- R29: value 220k -> 240k
- R45, R58: device rcl:R-EU_R0805 -> rcl:R-EU_M0805
Other:
- note added: "?"
- note added: "Display doesn't have a very strong pulldown resistor."
- note added: "For 7 pins, the PN is the same as PWM connector. 6-PIN is the default PN: 1516282"
