File: eagle/ftdi.brd (EAGLE design)
At the start: 48 x 28 mm, 34 parts, among them IC1 FT232RL, Q1 BCX70SMD, T5 BC847, T6 BC847, U1 SN65HVD1780

Commit message: Strain sensor with signed ad value, highest gain. Averaging moved, produced aliasing issues. Bootloader dind;t want to stay in bootload mode. Removed hex files from commit. Bom added
Parts:
- R32: value 1k -> 4k7
Changed lines of the file:
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@@
 <attribute name="VALUE" x="39.37" y="2.54" size="1.27" layer="27"/>
 </element>
-<element name="R32" library="rcl" package="M0805" value="1k" x="40.64" y="7.62" smashed="yes" rot="R180">
+<element name="R32" library="rcl" package="M0805" value="4k7" x="40.64" y="7.62" smashed="yes" rot="R180">
 <attribute name="NAME" x="37.7825" y="9.04875" size="1.016" layer="25" rot="R270"/>
 <attribute name="VALUE" x="41.91" y="10.16" size="1.27" layer="27" rot="R180"/>
