File: eagle/ftdi.sch (EAGLE design)
At the start: 34 parts, among them IC1 FT232RL, Q1 BCX70SMD, T5 BC847, T6 BC847, U1 SN65HVD1780

Commit message: Strain sensor with signed ad value, highest gain. Averaging moved, produced aliasing issues. Bootloader dind;t want to stay in bootload mode. Removed hex files from commit. Bom added
Parts:
- R32: value 1k -> 4k7
Other:
- note added: "Mount 1k ~ 4.7k pullup resistor for 5V data standalone"
- note removed: "Mount 1k resistor for 5V data standalone"
Changed lines of the file:
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@@
 <part name="R30" library="rcl" deviceset="R-EU_" device="M0805" value="1k"/>
 <part name="R31" library="rcl" deviceset="R-EU_" device="M0805" value="10R"/>
-<part name="R32" library="rcl" deviceset="R-EU_" device="M0805" value="1k"/>
+<part name="R32" library="rcl" deviceset="R-EU_" device="M0805" value="4k7"/>
 <part name="R33" library="rcl" deviceset="R-EU_" device="M0805" value="390k"/>
 <part name="R34" library="rcl" deviceset="R-EU_" device="M0805" value="100k"/>
@@
 <text x="205.74" y="144.78" size="1.778" layer="97">For one wire: Only use PIN1.</text>
 <text x="205.74" y="142.24" size="1.778" layer="97">For start board: 2 wires, host has an opto output.</text>
-<text x="12.7" y="312.42" size="1.778" layer="97">Mount 1k resistor for 5V data standalone</text>
+<text x="12.7" y="312.42" size="1.778" layer="97">Mount 1k ~ 4.7k pullup resistor for 5V data standalone</text>
 <text x="10.16" y="101.6" size="1.778" layer="97" rot="R180">Select 5V IO or 3V3 IO</text>
 <text x="284.48" y="195.58" size="1.778" layer="97">EDIT: Do this with 2 NPN's instead of sinking.</text>
